File: pc_power_control.kicad_sch (KiCad schematic)
At the start: 16 parts, among them IC1 NSVBC847BDW1T2G, J1 JFP1, J2 Conn_Serial, SW1 Reset, SW2 Flash, U1 ESP-12E

Commit message: fixed button pin assignment
Connections:
- net gpio0: now also SW2.3 (B); no longer SW2.2 (B)
- net at R1.2, U1.1 (~{RST}): now also SW1.3 (B); no longer SW1.2 (B)
Other:
- company: (none) -> Florian Hye
- title: (none) -> PC Power Control
Changed lines of the file:
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@@
 (kicad_sch (version 20230121) (generator eeschema)
   (paper "A4")
+  (title_block
+    (title "PC Power Control")
+    (date "2023-10-31")
+    (rev "1.2")
+    (company "Florian Hye")
+  )
   (junction (at 133.35 100.33) (diameter 0) (color 0 0 0 0)
   )
@@
     )
   )
-  (symbol (lib_id "Switch:SW_SPST") (at 74.93 54.61 0) (unit 1)
+  (symbol (lib_name "SW_SPST_1") (lib_id "Switch:SW_SPST") (at 74.93 54.61 0) (unit 1)
     (in_bom yes) (on_board yes) (dnp no) (fields_autoplaced)
     (property "Reference" "SW1" (at 74.93 48.26 0)
@@
       (effects (font (size 1.27 1.27)))
     )
-    (property "Footprint" "Samacsys:RKC2SJF170SMTRLFS" (at 74.93 54.61 0)
+    (property "Footprint" "Samacsys:RKC2SJF170SMTRLFS" (at 74.93 57.15 0)
       (effects (font (size 1.27 1.27)) hide)
     )
@@
     )
     (pin "1")
-    (pin "2")
+    (pin "3")
     (instances
       (project "pc_power_control"
@@
       (effects (font (size 1.27 1.27)))
     )
-    (property "Footprint" "Samacsys:RKC2SJF170SMTRLFS" (at 54.61 74.93 0)
+    (property "Footprint" "Samacsys:RKC2SJF170SMTRLFS" (at 54.61 77.47 0)
       (effects (font (size 1.27 1.27)) hide)
     )
@@
     )
     (pin "1")
-    (pin "2")
-    (instances
-      (project "pc_power_control"
+    (pin "3")
+    (instances
+      (project "pc_power_control"
